File: sr32gpo.kicad_sch (KiCad schematic)
At the start: 67 parts

Commit message: Redo with updated SOIC-16 footprint, better GND planes, and tentative fields for PCBWay assembly. Unverified.
Parts:
- C1, C2, C3, C4: value (none) -> 100n; footprint (none) -> Capacitor_SMD:C_0603_1608Metric
- C5: value (none) -> 10u; footprint (none) -> Capacitor_SMD:C_0805_2012Metric_Pad1.18x1.45mm_HandSolder
- H1, H2, H3, H4: value (none) -> ~; footprint (none) -> MountingHole:MountingHole_3mm_Pad
- J1: value (none) -> Power; footprint (none) -> TerminalBlock:TerminalBlock_bornier-2_P5.08mm
- J11, J12, J21, J22, J31, J32, J41, J42: value (none) -> GPO; footprint (none) -> Connectors:1X08
- J13, J23, J33, J43: value (none) -> GND; footprint (none) -> Connectors:1X08
- J2, J3, J4, J5: value (none) -> Power; footprint (none) -> Connector_PinHeader_2.54mm:PinHeader_1x02_P2.54mm_Vertical
- J6, J7: value (none) -> Data; footprint (none) -> Connector_PinHeader_2.54mm:PinHeader_1x06_P2.54mm_Vertical
- JP1: value (none) -> ~OESEL; footprint (none) -> Connector_PinHeader_2.54mm:PinHeader_1x03_P2.54mm_Vertical
- R1, R11, R12, R13, R14, R15, R16, R17, R18, R21, R22, R23, R24, R25, R26, R27, R28, R31, R32, R33, R34, R35, R36, R37, R38, R41, R42, R43, R44, R45, R46, R47, R48: value (none) -> 4.7k; footprint (none) -> Resistor_SMD:R_0603_1608Metric
- U1, U2, U3, U4: value (none) -> 74HC595; footprint (none) -> Package_SO:SOIC-16_3.9x9.9mm_P1.27mm
- U11: value (none) -> LD1117V33; footprint (none) -> Package_TO_SOT_SMD:SOT-223-3_TabPin2

Commit message: Update to KiCad v8, improve silkscreen, generate BOM and POS files for PCBWay
Parts:
- C1, C2, C3, C4: LCSC C14663 -> (none)
- C5: footprint Capacitor_SMD:C_0805_2012Metric_Pad1.18x1.45mm_HandSolder -> Capacitor_SMD:C_0805_2012Metric
- H1, H2, H3, H4, JP1: now not fitted; now left out of the parts list
- J1, J2, J3, J4, J5: symbol Connector:Conn_01x02_Male -> Connector:Conn_01x02_Pin; now not fitted; now left out of the parts list
- J11, J12, J13, J21, J22, J23, J31, J32, J33, J41, J42, J43: footprint Connectors:1X08 -> Connector_PinHeader_2.54mm:PinHeader_1x08_P2.54mm_Vertical; symbol Connector:Conn_01x08_Female -> Connector:Conn_01x08_Socket; now not fitted; now left out of the parts list
- J6, J7: symbol Connector:Conn_01x06_Male -> Connector:Conn_01x06_Pin; now not fitted; now left out of the parts list
- R1, R11, R12, R13, R14, R15, R16, R17, R18, R21, R22, R23, R24, R25, R26, R27, R28, R31, R32, R33, R34, R35, R36, R37, R38, R41, R42, R43, R44, R45, R46, R47, R48: LCSC C23162 -> (none)
- U11: value LD1117V33 -> LD1117V50; symbol Ken:LD1117 -> Regulator_Linear:AP1117-50
